Commit message: Package renaming

File: sw_neuronbot2_gazebo/urdf/neuronbot2.urdf (robot description, URDF)
Before this commit: robot neuronbot2_gazebo/models/neuronbot2, 6 links, 5 joints
Links:
- link base_link: geometry collision box size=0.25 0.25 0.25; visual mesh filename=package://sw_neuronbot2_gazebo/models/neuronbot2/meshes/neu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 scale=0.001 0.001 0.001
- link laser_frame: geometry collision mesh filename=package://sw_neuronbot2_gazebo/models/neuronbot2/meshes/neu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 scale=0.001 0.001 0.001; visual mesh filename=package://sw_neuronbot2_gazebo/models/neuronbot2/meshes/neu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 scale=0.001 0.001 0.001
- link wheel_left_link: geometry collision mesh filename=package://sw_neuronbot2_gazebo/models/neuronbot2/meshes/neu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 scale=0.001 0.001 0.001; visual mesh filename=package://sw_neuronbot2_gazebo/models/neuronbot2/meshes/neu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 scale=0.001 0.001 0.001
- link wheel_right_link: geometry collision mesh filename=package://sw_neuronbot2_gazebo/models/neuronbot2/meshes/neu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 scale=0.001 0.001 0.001; visual mesh filename=package://sw_neuronbot2_gazebo/models/neuronbot2/meshes/neu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 scale=0.001 0.001 0.001
